Commit message: add pid debugger

File: FlightEnv/assets/250.urdf (robot description, URDF)
Before this commit: robot cf2, 6 links, 5 joints
Links:
- link base_link: mass 0.616 -> 0.452

Commit message: 6.4

File: FlightEnv/assets/250.urdf (robot description, URDF)
Before this commit: robot cf2, 6 links, 5 joints
Links:
- link base_link: geometry collision cylinder length=.094 radius=.15; visual cylinder length=0.025 radius=0.2
